File: pcb/zynq_test/ZynqPWR+Config.kicad_sch (KiCad schematic)
At the start: 43 parts, among them SW601 PS_RST, SW602 PROG, U202 XC7Z020-2CLG400I

Commit message: Version sent to JLCPCB
Parts:
- C601, C604, C605, C632: JLCPCB Part# (none) -> C23742; PART_NUMBER (none) -> CL32A107MPVNNNE
- C602, C607, C608, C609, C610, C612, C627, C628, C630, C631: JLCPCB Part# (none) -> C23733; PART_NUMBER (none) -> CL05A475MP5NRNC
- C603, C619: JLCPCB Part# (none) -> C525654; PART_NUMBER (none) -> CL32A476KPJNNNE
- C606, C611, C613, C614, C615, C616, C617, C618, C620, C621, C622, C623, C624, C625, C626: JLCPCB Part# (none) -> C88946; PART_NUMBER (none) -> GRM155R71A474KE01D
- C629: JLCPCB Part# (none) -> C1525; PART_NUMBER (none) -> CL05B104KO5NNNC
- C633: JLCPCB Part# (none) -> C528969; PART_NUMBER (none) -> GRM32ER60G337ME05L
- D601: JLCPCB Part# (none) -> C192672; PART_NUMBER (none) -> TJ-S2012SW8TGLC7K-A5
- L601: JLCPCB Part# (none) -> C5120901; PART_NUMBER (none) -> 742792023
- R601, R603: JLCPCB Part# (none) -> C327817; PART_NUMBER (none) -> MR04X4701FTL
- R602: JLCPCB Part# (none) -> C191123; PART_NUMBER (none) -> ERJ2RKF1002X
- R604, R605: JLCPCB Part# (none) -> C412979; PART_NUMBER (none) -> ERJ2GEJ221X
- SW601, SW602: JLCPCB Part# (none) -> C5769038; PART_NUMBER (none) -> MJTP1243
- U202: JLCPCB Part# (none) -> C569043; PART_NUMBER (none) -> XC7Z020-2CLG400I
