File: pcb/zynq_test/CAMERA_TX.kicad_sch (KiCad schematic)
At the start: 42 parts, among them J1701 SFW15R-2STE1LF, U1701 SN75DPHY440, U1702 TCA9406DC

Commit message: Version sent to JLCPCB
Parts:
- C1701, C1702, C1703, C1704, C1706, C1707: JLCPCB Part# (none) -> C1525; PART_NUMBER (none) -> CL05B104KO5NNNC
- C1705: JLCPCB Part# (none) -> C525654; PART_NUMBER (none) -> CL32A476KPJNNNE
- J1701: JLCPCB Part# (none) -> C3167933; PART_NUMBER (none) -> SFW15R-2STE1LF
- R1701, R1704, R1705, R1708, R1709, R1712: JLCPCB Part# (none) -> C6491855; PART_NUMBER (none) -> AC0402FR-7W60R4L
- R1702, R1703, R1706, R1707, R1710, R1711: JLCPCB Part# (none) -> C412976; PART_NUMBER (none) -> ERJ2GEJ151X
- R1713, R1714, R1715, R1716, R1717, R1718: JLCPCB Part# (none) -> C412974; PART_NUMBER (none) -> ERJ2GEJ121X
- R1719, R1720, R1730, R1731: PART_NUMBER (none) -> ERJ2GEJ162X
- R1721, R1723: JLCPCB Part# (none) -> C412995; PART_NUMBER (none) -> ERJ2GEJ162X
- R1722, R1724, R1725, R1726, R1727, R1728: PART_NUMBER (none) -> ERJ2RKF1002X
- R1729: value 1k0 -> 1k; JLCPCB Part# (none) -> C242161; PART_NUMBER (none) -> ERJ2RKF1001X
- U1701: JLCPCB Part# (none) -> C2863793; PART_NUMBER (none) -> SN75DPHY440SSRHRR
- U1702: JLCPCB Part# (none) -> C840107; PART_NUMBER (none) -> TCA9406DCUR
