File: pcb/zynq_test/RX_camera.kicad_sch (KiCad schematic)
At the start: 33 parts, among them J1501 SFW15R-2STE1LF, U1501 TCA9406DC, U1502 SN75DPHY440

Commit message: Version sent to JLCPCB
Parts:
- C1501, C1502, C1503, C1504, C1505, C1507: JLCPCB Part# (none) -> C1525; PART_NUMBER (none) -> CL05B104KO5NNNC
- C1506: JLCPCB Part# (none) -> C525654; PART_NUMBER (none) -> CL32A476KPJNNNE
- J1501: JLCPCB Part# (none) -> C3167933; PART_NUMBER (none) -> SFW15R-2STE1LF
- R1501, R1502, R1503, R1504, R1505, R1506: JLCPCB Part# (none) -> C159871; PART_NUMBER (none) -> RK73B1ETTP101J
- R1507, R1508, R1509: JLCPCB Part# (none) -> C412976; PART_NUMBER (none) -> ERJ2GEJ151X
- R1510, R1514: JLCPCB Part# (none) -> C412995; PART_NUMBER (none) -> ERJ2GEJ162X
- R1511, R1515, R1517, R1518, R1521, R1522: PART_NUMBER (none) -> ERJ2RKF1002X
- R1512, R1513, R1519, R1520: PART_NUMBER (none) -> ERJ2GEJ162X
- R1516: value 1k0 -> 1k; JLCPCB Part# (none) -> C242161; PART_NUMBER (none) -> ERJ2RKF1001X
- U1501: JLCPCB Part# (none) -> C840107; PART_NUMBER (none) -> TCA9406DCUR
- U1502: JLCPCB Part# (none) -> C2863793; PART_NUMBER (none) -> SN75DPHY440SSRHRR
