File: pcb/zynq_test/programmer.kicad_sch (KiCad schematic)
At the start: 43 parts, among them J701 Conn_01x06_Pin, J702 USB_B_Micro, U701 ESD8104, U702 FT2232HQ, U703 DSC1001CI2-012, U704 93LCxxB, U705 ESD8104, U706 74AUC1G07

Commit message: Version sent to JLCPCB
Parts:
- C701, C702, C703, C704, C705, C706, C707, C708, C709, C710, C713: JLCPCB Part# (none) -> C1525; PART_NUMBER (none) -> CL05B104KO5NNNC
- C711, C712: JLCPCB Part# (none) -> C23733; PART_NUMBER (none) -> CL05A475MP5NRNC
- J701: now left out of the parts list
- J702: JLCPCB Part# (none) -> C132562; PART_NUMBER (none) -> 10118193-0001LF
- L701, L702: JLCPCB Part# (none) -> C5120901; PART_NUMBER (none) -> 742792023
- R701, R702, R715, R718, R720: JLCPCB Part# (none) -> C191123; PART_NUMBER (none) -> ERJ2RKF1002X
- R703, R704, R705, R706: JLCPCB Part# (none) -> C159964; PART_NUMBER (none) -> RK73H1ETTP22R0F
- R707, R708, R709, R710, R711, R712, R713, R716: JLCPCB Part# (none) -> C242160; PART_NUMBER (none) -> ERJ2GE0R00X
- R714: JLCPCB Part# (none) -> C242161; PART_NUMBER (none) -> ERJ2RKF1001X
- R717: JLCPCB Part# (none) -> C363271; PART_NUMBER (none) -> HPCR0402F12K0K9
- R719: JLCPCB Part# (none) -> C159880; PART_NUMBER (none) -> RK73B1ETTP202J
- U701, U705: JLCPCB Part# (none) -> C94394; PART_NUMBER (none) -> ESD8104MUTAG
- U702: JLCPCB Part# (none) -> C3025148; PART_NUMBER (none) -> FT2232HQ-TRAY
- U703: JLCPCB Part# (none) -> C611391; PART_NUMBER (none) -> DSC1001CI2-012.0000
- U704: JLCPCB Part# (none) -> C1348804; PART_NUMBER (none) -> 93LC46B/SN
- U706: JLCPCB Part# (none) -> C163714; PART_NUMBER (none) -> SN74AUC1G07DBVR
Connections:
- net +3V3: now also J701.6 (Pin_6)
- no-connect marks 33 -> 32
Other:
- note removed: "6 is for PWR we don't want power"
